File: hardware/carrier/carrier.kicad_pcb (KiCad board)
At the start: 2 copper layers, 112 x 65.9 mm, 47 parts, among them J1 B6252HB, J2 B6252HB, J3 B6252HB, SW1-1 SW_Push_DPDT, SW1-2 SW_Push_DPDT, SW4 SW_Push_DPDT, SW5 SW_Push_DPDT, U1 Pico

Commit message: update (channel can chenge)
Parts:
- C1, C12, C13, C4: value 1uf -> 100nf
- R16, R8: value 100k -> 40k
- moved D4 8.11 mm to (106.0, 91.4), turned to -90 degrees
- moved D3 2.74 mm to (108.8, 99.0)
Routing:
- net adc3: track 146.4 -> 117.7 mm
- net +3.3VADC: track 274.4 -> 271.1 mm
