File: hardware/carrier/carrier.kicad_sch (KiCad schematic)
At the start: 47 parts, among them J1 B6252HB, J2 B6252HB, J3 B6252HB, SW1-1 SW_Push_DPDT, SW1-2 SW_Push_DPDT, SW4 SW_Push_DPDT, SW5 SW_Push_DPDT, U1 Pico

Commit message: update (channel can chenge)
Parts:
- C1, C12, C13, C4: value 1uf -> 100nf
- R16, R8: value 100k -> 40k
Changed lines of the file:
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@@
       (effects (font (size 1.27 1.27)))
     )
-    (property "Value" "1uf" (at 124.46 156.21 90)
+    (property "Value" "100nf" (at 124.46 156.21 90)
       (effects (font (size 1.27 1.27)))
     )
@@
       (effects (font (size 1.27 1.27)) (justify left))
     )
-    (property "Value" "100k" (at 54.61 63.5 0)
+    (property "Value" "40k" (at 54.61 63.5 0)
       (effects (font (size 1.27 1.27)) (justify left))
     )
@@
       (effects (font (size 1.27 1.27)))
     )
-    (property "Value" "1uf" (at 87.63 50.8 90)
+    (property "Value" "100nf" (at 87.63 50.8 90)
       (effects (font (size 1.27 1.27)))
     )
@@
       (effects (font (size 1.27 1.27)))
     )
-    (property "Value" "1uf" (at 67.31 104.14 90)
+    (property "Value" "100nf" (at 67.31 104.14 90)
       (effects (font (size 1.27 1.27)))
     )
@@
       (effects (font (size 1.27 1.27)))
     )
-    (property "Value" "1uf" (at 166.37 64.77 90)
+    (property "Value" "100nf" (at 166.37 64.77 90)
       (effects (font (size 1.27 1.27)))
     )
@@
       (effects (font (size 1.27 1.27)) (justify left))
     )
-    (property "Value" "100k" (at 129.54 77.47 0)
-      (effects (font (size 1.27 1.27)) (justify left))
-    )
+    (property "Value" "40k" (at 129.54 77.47 0)
+      (effects (font (size 1.27 1.27)) (justify left))
+    )
