File: hardware/v2/analog/analog.kicad_sch (KiCad schematic)
At the start: 24 parts, among them J1 Conn_Coaxial, K1 Relay_SPDT, Q1 BC547, U1 CD4051B, U2 TL081, U3 TL431LP

Commit message: update
Parts:
- R13: value 100K -> 3k
Changed lines of the file:
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@@
       (effects (font (size 1.27 1.27)))
     )
-    (property "Value" "100K" (at 67.31 26.67 90)
+    (property "Value" "3k" (at 67.31 26.67 90)
       (effects (font (size 1.27 1.27)))
     )
