File: hardware/v2/analog/analog.kicad_pcb (KiCad board)
At the start: 2 copper layers, 4 parts, among them Q1 BC547, U3 TL431LP

Commit message: update
Parts:
- added Q2: BC547, Package_TO_SOT_THT:TO-92_Inline, F.Cu at (115.0, 55.7)
- added Q3: BC557, Package_TO_SOT_THT:TO-92_Inline, F.Cu at (115.0, 61.5)
Connections:
- net adc renamed ADC
- U3 pad 1: unconnected-(U3-REF-Pad1) -> Net-(U3-REF)
- U3 pad 2: unconnected-(U3-A-Pad2) -> GND
- U3 pad 3: unconnected-(U3-K-Pad3) -> Net-(Q2-B)

Commit message: update
Parts:
- added C1: C, Capacitor_THT:C_Disc_D6.0mm_W2.5mm_P5.00mm, F.Cu at (-52.0, 197.1)
- added C2: 10pf 1kv, Capacitor_THT:C_Disc_D7.5mm_W5.0mm_P7.50mm, F.Cu at (-68.5, 220.8)
- added C3: 100pf, Capacitor_THT:C_Disc_D7.5mm_W5.0mm_P7.50mm, F.Cu at (-68.5, 227.3)
- added C4: 100nF, Capacitor_THT:C_Disc_D7.5mm_W5.0mm_P7.50mm, F.Cu at (450.9, 138.5)
- added C5: 100nF, Capacitor_THT:C_Disc_D7.5mm_W5.0mm_P7.50mm, F.Cu at (403.9, 137.2)
- added C6: 100nf, Capacitor_THT:C_Disc_D7.5mm_W2.5mm_P5.00mm, F.Cu at (426.7, 15.4)
- added C7: 47uF, Capacitor_THT:C_Disc_D7.5mm_W5.0mm_P7.50mm, F.Cu at (457.2, 30.6)
- added C8: 100nf, Capacitor_THT:C_Disc_D7.5mm_W2.5mm_P5.00mm, F.Cu at (459.7, 16.6)
- added C9: 220uF, Capacitor_THT:CP_Radial_D10.0mm_P5.00mm, F.Cu at (475.0, 31.8)
- added D3: 1n4148, Diode_THT:D_DO-35_SOD27_P7.62mm_Horizontal, F.Cu at (429.3, 36.8)
- added D4: 1n4148, Diode_THT:D_DO-35_SOD27_P7.62mm_Horizontal, F.Cu at (433.1, 25.4)
- added D5: 1n4148, Diode_THT:D_DO-35_SOD27_P7.62mm_Horizontal, F.Cu at (449.6, 26.7)
- added D6: 1n4148, Diode_THT:D_DO-35_SOD27_P7.62mm_Horizontal, F.Cu at (463.6, 25.4)
- added J1: Conn_Coaxial, Connector_Coaxial:BNC_Amphenol_B6252HB-NPP3G-50_Horizontal, F.Cu at (143.5, 139.7)
- added K2: SANYOU_SRD_Form_C, Relay_THT:Relay_SPDT_SANYOU_SRD_Series_Form_C, F.Cu at (-112.0, 188.6)
- added Q4: BC547, Package_TO_SOT_THT:TO-92_Inline, F.Cu at (414.0, 11.4)
- added Q5: BC557, Package_TO_SOT_THT:TO-92_Inline, F.Cu at (414.0, 21.6)
- added R1: 128k, Resistor_THT:R_Axial_DIN0309_L9.0mm_D3.2mm_P12.70mm_Horizontal, F.Cu at (-37.5, 19.7)
- added R10: 1k, Resistor_THT:R_Axial_DIN0309_L9.0mm_D3.2mm_P12.70mm_Horizontal, F.Cu at (-37.5, 62.5)
- added R11: 1M, Resistor_THT:R_Axial_DIN0309_L9.0mm_D3.2mm_P12.70mm_Horizontal, F.Cu at (-84.6, 229.8)
- added R12: 100K, Resistor_THT:R_Axial_DIN0309_L9.0mm_D3.2mm_P12.70mm_Horizontal, F.Cu at (-84.6, 234.6)
- added R13: 1K, Resistor_THT:R_Axial_DIN0309_L9.0mm_D3.2mm_P12.70mm_Horizontal, F.Cu at (108.6, 161.3)
- added R14: 1K, Resistor_THT:R_Axial_DIN0309_L9.0mm_D3.2mm_P12.70mm_Horizontal, F.Cu at (426.7, 120.7)
- added R15: 62K, Resistor_THT:R_Axial_DIN0309_L9.0mm_D3.2mm_P12.70mm_Horizontal, F.Cu at (415.3, 157.5)
- added R16: 20K, Resistor_THT:R_Axial_DIN0309_L9.0mm_D3.2mm_P12.70mm_Horizontal, F.Cu at (419.1, 139.7)
- added R17: 10k, Resistor_THT:R_Axial_DIN0309_L9.0mm_D3.2mm_P12.70mm_Horizontal, F.Cu at (481.3, 10.2)
- added R18: 10k, Resistor_THT:R_Axial_DIN0309_L9.0mm_D3.2mm_P12.70mm_Horizontal, F.Cu at (481.3, 25.4)
- added R2: 64k, Resistor_THT:R_Axial_DIN0309_L9.0mm_D3.2mm_P12.70mm_Horizontal, F.Cu at (-37.5, 24.5)
- added R3: 32k, Resistor_THT:R_Axial_DIN0309_L9.0mm_D3.2mm_P12.70mm_Horizontal, F.Cu at (-37.5, 29.2)
- added R4: 16k, Resistor_THT:R_Axial_DIN0309_L9.0mm_D3.2mm_P12.70mm_Horizontal, F.Cu at (-37.5, 34.0)
- added R5: 8k, Resistor_THT:R_Axial_DIN0309_L9.0mm_D3.2mm_P12.70mm_Horizontal, F.Cu at (-37.5, 38.7)
- added R6: 10k, Resistor_THT:R_Axial_DIN0309_L9.0mm_D3.2mm_P12.70mm_Horizontal, F.Cu at (101.0, -132.4)
- added R7: 10k, Resistor_THT:R_Axial_DIN0309_L9.0mm_D3.2mm_P12.70mm_Horizontal, F.Cu at (101.0, -127.6)
- added R8: 4k, Resistor_THT:R_Axial_DIN0309_L9.0mm_D3.2mm_P12.70mm_Horizontal, F.Cu at (-37.5, 53.0)
- added R9: 2k, Resistor_THT:R_Axial_DIN0309_L9.0mm_D3.2mm_P12.70mm_Horizontal, F.Cu at (-37.5, 57.7)
- added TP1: 1khz, TestPoint:TestPoint_Pad_3.0x3.0mm, F.Cu at (259.7, 50.9)
- added TP2: GNDA, TestPoint:TestPoint_Pad_3.0x3.0mm, F.Cu at (259.7, 55.9)
- added TP3: 3v3, TestPoint:TestPoint_Pad_3.0x3.0mm, F.Cu at (259.7, 61.0)
- added U1: CD4051B, Package_DIP:DIP-8_W7.62mm_LongPads, F.Cu at (115.4, 99.1)
- added U2: TL081, Package_DIP:DIP-8_W7.62mm_LongPads, F.Cu at (127.0, 99.1)
- added U4: Pico, MCU_RaspberryPi_and_Boards:RPi_Pico_SMD_TH, F.Cu at (175.3, 118.1)
- moved Q3 335.9 mm to (440.7, 143.5), turned to 90 degrees
- moved Q2 333.7 mm to (440.7, 128.3), turned to -90 degrees
- moved U3 323.6 mm to (396.2, 152.4), turned to 90 degrees
- moved D1 212.4 mm to (103.4, -146.4)
- moved D2 212.4 mm to (103.4, -142.8)
- moved Q1 91.5 mm to (113.7, 153.0)
Connections:
- net ADC renamed pico-adc
- D1 pad 1: +3.3V -> +3.3VA
- D2 pad 2: GND -> GNDA
- Q2 pad 3: 3V3_REF -> +3.3VA
- Q3 pad 3: 3V3_REF -> +3.3VA
Other:
- board outline added: 127 x 76.2 mm

Commit message: update 2
Parts:
- moved TP1 81.6 mm to (196.8, 102.9)
- moved TP2 81.6 mm to (196.8, 107.9)
- moved TP3 81.6 mm to (196.8, 113.0)
Changed lines of the file:
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@@
 	(footprint "TestPoint:TestPoint_Pad_3.0x3.0mm"
 		(layer "F.Cu")
-		(at 259.715 60.96)
+		(at 196.85 112.97)
 		(descr "SMD rectangular pad as test Point, square 3.0mm side length")
 		(tags "test point SMD pad rectangle square")
@@
 	(footprint "TestPoint:TestPoint_Pad_3.0x3.0mm"
 		(layer "F.Cu")
-		(at 259.715 50.86)
+		(at 196.85 102.87)
 		(descr "SMD rectangular pad as test Point, square 3.0mm side length")
 		(tags "test point SMD pad rectangle square")
@@
 	(footprint "TestPoint:TestPoint_Pad_3.0x3.0mm"
 		(layer "F.Cu")
-		(at 259.715 55.91)
+		(at 196.85 107.92)
 		(descr "SMD rectangular pad as test Point, square 3.0mm side length")
 		(tags "test point SMD pad rectangle square")
